Commit message: urdf limit

File: mra7a_description/urdf/mra7a_autogenerated_from_xacro.urdf (robot description, URDF)
Before this commit: robot mra7a, 11 links, 10 joints
Joints:
- joint Joint2: limit lower=-2.35 upper=2.35 effort=90 velocity=1.31 -> lower=-2.18 upper=2.18 effort=90 velocity=1.31
- joint Joint4: limit lower=-2.35 upper=2.35 effort=67 velocity=1.31 -> lower=-2.3 upper=2.3 effort=67 velocity=1.31
- joint Joint6: limit lower=-2.35 upper=2.35 effort=67 velocity=1.57 -> lower=-2.05 upper=2.05 effort=67 velocity=1.57
- joint fixed: origin xyz=0 0 0.5 rpy=0 0 0 -> xyz=0 0 0.0 rpy=0 0 0
